File: Composite Video Amplifier.sch (KiCad schematic (older format))
At the start: 15 parts, among them J1 Audio Input, J2 Video Input, J3 Output, Q1 2N3904, Q2 2N3906

Commit message: Fixed electrical checks
Parts:
- J2: symbol Conn_01x05 -> Video_IN
Changed lines of the file:
@@
 LIBS:contrib
 LIBS:valves
+LIBS:ports
+LIBS:Composite Video Amplifier-cache
 EELAYER 25 0
 EELAYER END
@@
 $EndDescr
 $Comp
-L Conn_01x05 J2
+L Video_IN J2
 U 1 1 5C1246EF
 P 3925 4150

Commit message: PCB layout done
Parts:
- removed J1: Audio Input, Pin_Headers:Pin_Header_Straight_1x02_Pitch2.54mm, symbol Conn_01x02
- removed J2: Video Input, Pin_Headers:Pin_Header_Straight_1x05_Pitch2.54mm, symbol Video_IN
- added J1: Video, Pin_Headers:Pin_Header_Straight_1x04_Pitch2.54mm, symbol Video
- J2: renamed from J3; symbol Conn_01x04 -> Output
Connections:
- net AUD_IN: now also R8.1, J1.3 (Pin_2); no longer R8.2
- net AUD_OUT: now also R8.2; no longer R8.1
- net GND: now also R3.1, R5.1, R7.1, J1.4 (Pin_1); no longer R3.2, R5.2, R7.2
- net VCC: now also J1.1 (Pin_4)
- net VID_IN: now also R1.1, J1.2 (Pin_3); no longer R1.2
- net VID_OUT: now also R7.2; no longer R7.1
- net at C1.1, RV1.2, RV1.3: now also R1.2; no longer R1.1
- net at Q1.2 (B), R2.2, RV1.1: now also R3.2; no longer R3.1
- net at Q1.1 (E): now also R5.2; no longer R5.1
- no-connect marks 2 -> 0
Other:
- moved on the sheet: R8
Changed lines of the file:
@@
 $EndDescr
-$Comp
-L Video_IN J2
-U 1 1 5C1246EF
-P 3925 4150
-F 0 "J2" H 3925 4450 50  0000 C CNN
-F 1 "Video Input" H 3925 3850 50  0000 C CNN
-F 2 "Pin_Headers:Pin_Header_Straight_1x05_Pitch2.54mm" H 3925 4150 50  0001 C CNN
-F 3 "" H 3925 4150 50  0001 C CNN
-	1    3925 4150
-	-1   0    0    1
-$EndComp
 $Comp
 L GND #PWR01
 U 1 1 5C124730
-P 4200 4425
-F 0 "#PWR01" H 4200 4175 50  0001 C CNN
-F 1 "GND" H 4200 4275 50  0000 C CNN
-F 2 "" H 4200 4425 50  0001 C CNN
-F 3 "" H 4200 4425 50  0001 C CNN
-	1    4200 4425
-	1    0    0    -1
-$EndComp
-Wire Wire Line
-	4200 4425 4200 4350
-Wire Wire Line
-	4200 4350 4125 4350
+P 4200 4325
+F 0 "#PWR01" H 4200 4075 50  0001 C CNN
+F 1 "GND" H 4200 4175 50  0000 C CNN
+F 2 "" H 4200 4325 50  0001 C CNN
+F 3 "" H 4200 4325 50  0001 C CNN
+	1    4200 4325
+	1    0    0    -1
+$EndComp
 $Comp
 L VCC #PWR02
@@
 $EndComp
 Wire Wire Line
-	4200 3875 4200 4150
-Wire Wire Line
-	4200 4150 4125 4150
-Wire Wire Line
 	4125 4050 4650 4050
-Text Label 4225 4050 0    60   ~ 0
+Text Label 4125 4050 0    60   ~ 0
 VID_IN
 $Comp
@@
 F 3 "" H 4800 4050 50  0001 C CNN
 	1    4800 4050
-	0    1    1    0
+	0    -1   -1   0
 $EndComp
 Wire Wire Line
@@
 F 3 "" H 5475 4275 50  0001 C CNN
 	1    5475 4275
-	1    0    0    -1
+	-1   0    0    1
 $EndComp
 Wire Wire Line
@@
 F 3 "" H 5850 4475 50  0001 C CNN
 	1    5850 4475
-	1    0    0    -1
+	-1   0    0    1
 $EndComp
 Wire Wire Line
@@
 	5850 4625 5850 4775
 Wire Wire Line
-	5475 4700 7300 4700
+	5475 4700 7225 4700
 Connection ~ 5850 4700
 $Comp
@@
 F 3 "" H 6450 4275 50  0001 C CNN
 	1    6450 4275
-	1    0    0    -1
+	-1   0    0    1
 $EndComp
 Wire Wire Line
 	6450 3975 6450 4125
-Wire Wire Line
-	6450 4050 7375 4050
 Connection ~ 6450 4050
 Wire Wire Line
 	6450 4700 6450 4425
-$Comp
-L Conn_01x02 J1
-U 1 1 5C125EFF
-P 3925 2725
-F 0 "J1" H 3925 2825 50  0000 C CNN
-F 1 "Audio Input" H 3925 2525 50  0000 C CNN
-F 2 "Pin_Headers:Pin_Header_Straight_1x02_Pitch2.54mm" H 3925 2725 50  0001 C CNN
-F 3 "" H 3925 2725 50  0001 C CNN
-	1    3925 2725
-	-1   0    0    1
-$EndComp
-$Comp
-L GND #PWR05
-U 1 1 5C126148
-P 4200 2800
-F 0 "#PWR05" H 4200 2550 50  0001 C CNN
-F 1 "GND" H 4200 2650 50  0000 C CNN
-F 2 "" H 4200 2800 50  0001 C CNN
-F 3 "" H 4200 2800 50  0001 C CNN
-	1    4200 2800
-	1    0    0    -1
-$EndComp
-Wire Wire Line
-	4200 2800 4200 2725
-Wire Wire Line
-	4200 2725 4125 2725
 $Comp
 L R R8
 U 1 1 5C12628A
-P 4800 2625
-F 0 "R8" V 4880 2625 50  0000 C CNN
-F 1 "10k" V 4800 2625 50  0000 C CNN
-F 2 "Resistors_THT:R_Axial_DIN0207_L6.3mm_D2.5mm_P10.16mm_Horizontal" V 4730 2625 50  0001 C CNN
-F 3 "" H 4800 2625 50  0001 C CNN
-	1    4800 2625
-	0    1    1    0
-$EndComp
-Wire Wire Line
-	4125 2625 4650 2625
-NoConn ~ 4125 3950
-NoConn ~ 4125 4250
-$Comp
-L Conn_01x04 J3
+P 4800 5050
+F 0 "R8" V 4880 5050 50  0000 C CNN
+F 1 "10k" V 4800 5050 50  0000 C CNN
+F 2 "Resistors_THT:R_Axial_DIN0207_L6.3mm_D2.5mm_P10.16mm_Horizontal" V 4730 5050 50  0001 C CNN
+F 3 "" H 4800 5050 50  0001 C CNN
+	1    4800 5050
+	0    -1   -1   0
+$EndComp
+$Comp
+L Output J2
 U 1 1 5C1265F4
-P 7575 3950
-F 0 "J3" H 7575 4150 50  0000 C CNN
-F 1 "Output" H 7575 3650 50  0000 C CNN
-F 2 "Pin_Headers:Pin_Header_Straight_1x04_Pitch2.54mm" H 7575 3950 50  0001 C CNN
-F 3 "" H 7575 3950 50  0001 C CNN
-	1    7575 3950
+P 7575 4250
+F 0 "J2" H 7575 4450 50  0000 C CNN
+F 1 "Output" H 7575 3950 50  0000 C CNN
+F 2 "Pin_Headers:Pin_Header_Straight_1x04_Pitch2.54mm" H 7575 4250 50  0001 C CNN
+F 3 "" H 7575 4250 50  0001 C CNN
+	1    7575 4250
 	1    0    0    1
 $EndComp
@@
 VID_OUT
 Wire Wire Line
-	7375 3750 7300 3750
-Wire Wire Line
-	7300 3750 7300 2625
-Wire Wire Line
-	7300 2625 4950 2625
-Text Label 4200 2625 0    60   ~ 0
+	7300 5050 4950 5050
+Text Label 4125 4150 0    60   ~ 0
 AUD_IN
-Text Label 5100 2625 0    60   ~ 0
+Text Label 6675 5050 0    60   ~ 0
 AUD_OUT
-Wire Wire Line
-	7375 3950 7300 3950
-Wire Wire Line
-	7300 4700 7300 3850
 Connection ~ 6450 4700
-Wire Wire Line
-	7300 3850 7375 3850
-Connection ~ 7300 3950
 Text Notes 7025 6750 0    60   ~ 0
 Based on composite video modification for Atari 2600 by user simon.plata on AtariAge\nforums. Redesigned PCB to match my VDU projects.
+$Comp
+L Video J1
+U 1 1 5C129CEB
+P 3925 4150
+F 0 "J1" H 3925 4350 50  0000 C CNN
+F 1 "Video" H 3925 3850 50  0000 C CNN
+F 2 "Pin_Headers:Pin_Header_Straight_1x04_Pitch2.54mm" H 3925 4150 50  0001 C CNN
+F 3 "" H 3925 4150 50  0001 C CNN
+	1    3925 4150
+	-1   0    0    1
+$EndComp
+Wire Wire Line
+	4125 3950 4200 3950
+Wire Wire Line
+	4200 3950 4200 3875
+Wire Wire Line
+	4200 4250 4125 4250
+Wire Wire Line
+	4200 4250 4200 4325
+Wire Wire Line
+	6450 4050 7375 4050
+Wire Wire Line
+	7225 4150 7375 4150
+Wire Wire Line
+	4125 4150 4375 4150
+Wire Wire Line
+	4650 5050 4375 5050
+Wire Wire Line
+	4375 5050 4375 4150
+Wire Wire Line
+	7225 4700 7225 4150
+Wire Wire Line
+	7375 4250 7225 4250
+Connection ~ 7225 4250
+Wire Wire Line
+	7375 4350 7300 4350
+Wire Wire Line
+	7300 4350 7300 5050
 $EndSCHEMATC

Commit message: Improved silkscreen markings
Parts:
- C1: symbol C_Small -> Device:C_Small
- J1: symbol Video -> ports:Video
- J2: symbol Output -> ports:Output
- Q1: symbol 2N3904 -> Transistor_BJT:2N3904
- Q2: symbol 2N3906 -> Transistor_BJT:2N3906
- R1, R2, R3, R4, R5, R6, R7, R8: symbol R -> Device:R
- RV1: symbol POT -> Device:R_POT
Changed lines of the file:
@@
-EESchema Schematic File Version 2
-LIBS:power
-LIBS:device
-LIBS:switches
-LIBS:relays
-LIBS:motors
-LIBS:transistors
-LIBS:conn
-LIBS:linear
-LIBS:regul
-LIBS:74xx
-LIBS:cmos4000
-LIBS:adc-dac
-LIBS:memory
-LIBS:xilinx
-LIBS:microcontrollers
-LIBS:dsp
-LIBS:microchip
-LIBS:analog_switches
-LIBS:motorola
-LIBS:texas
-LIBS:intel
-LIBS:audio
-LIBS:interface
-LIBS:digital-audio
-LIBS:philips
-LIBS:display
-LIBS:cypress
-LIBS:siliconi
-LIBS:opto
-LIBS:atmel
-LIBS:contrib
-LIBS:valves
-LIBS:ports
-LIBS:Composite Video Amplifier-cache
-EELAYER 25 0
+EESchema Schematic File Version 4
+EELAYER 30 0
 EELAYER END
 $Descr A4 11693 8268
@@
 $EndDescr
 $Comp
-L GND #PWR01
+L power:GND #PWR01
 U 1 1 5C124730
 P 4200 4325
@@
 $EndComp
 $Comp
-L VCC #PWR02
+L power:VCC #PWR02
 U 1 1 5C124750
 P 4200 3875
@@
 $EndComp
 Wire Wire Line
-	4125 4050 4650 4050
+	4125 4050 4575 4050
 Text Label 4125 4050 0    60   ~ 0
 VID_IN
 $Comp
-L C_Small C1
+L Device:C_Small C1
 U 1 1 5C1247A9
 P 4800 3775
@@
 $EndComp
 $Comp
-L R R1
+L Device:R R1
 U 1 1 5C1247F7
 P 4800 4050
@@
 Connection ~ 4575 4050
 Wire Wire Line
-	4950 4050 5100 4050
-Wire Wire Line
-	5025 3775 5025 4275
+	4950 4050 5025 4050
+Wire Wire Line
+	5025 3775 5025 4050
 Wire Wire Line
 	5025 3775 4900 3775
 $Comp
-L POT RV1
+L Device:R_POT RV1
 U 1 1 5C1248A3
 P 5250 4050
@@
 	5250 4275 5250 4200
 Wire Wire Line
-	5400 4050 5550 4050
-$Comp
-L R R2
+	5400 4050 5475 4050
+$Comp
+L Device:R R2
 U 1 1 5C12499D
 P 5475 3825
@@
 $EndComp
 $Comp
-L R R3
+L Device:R R3
 U 1 1 5C1249E5
 P 5475 4275
@@
 $EndComp
 Wire Wire Line
-	5475 3975 5475 4125
+	5475 3975 5475 4050
 Connection ~ 5475 4050
 $Comp
-L GND #PWR03
+L power:GND #PWR03
 U 1 1 5C124AD3
 P 5850 4775
@@
 	5475 4425 5475 4700
 $Comp
-L 2N3904 Q1
+L Transistor_BJT:2N3904 Q1
 U 1 1 5C124B77
 P 5750 4050
@@
 $EndComp
 $Comp
-L VCC #PWR04
+L power:VCC #PWR04
 U 1 1 5C124C34
-P 5850 3050
-F 0 "#PWR04" H 5850 2900 50  0001 C CNN
-F 1 "VCC" H 5850 3200 50  0000 C CNN
-F 2 "" H 5850 3050 50  0001 C CNN
-F 3 "" H 5850 3050 50  0001 C CNN
-	1    5850 3050
+P 5475 3050
+F 0 "#PWR04" H 5475 2900 50  0001 C CNN
+F 1 "VCC" H 5475 3200 50  0000 C CNN
+F 2 "" H 5475 3050 50  0001 C CNN
+F 3 "" H 5475 3050 50  0001 C CNN
+	1    5475 3050
 	1    0    0    -1
 $EndComp
@@
 	5475 3125 5475 3675
 $Comp
-L R R4
+L Device:R R4
 U 1 1 5C124C99
 P 5850 3550
@@
 $EndComp
 $Comp
-L R R5
+L Device:R R5
 U 1 1 5C124D36
 P 5850 4475
@@
 $EndComp
 Wire Wire Line
-	5850 3700 5850 3850
+	5850 3700 5850 3775
 Wire Wire Line
 	5850 4250 5850 4325
 Wire Wire Line
-	5850 4625 5850 4775
-Wire Wire Line
-	5475 4700 7225 4700
+	5850 4625 5850 4700
+Wire Wire Line
+	5475 4700 5850 4700
 Connection ~ 5850 4700
 $Comp
-L 2N3906 Q2
+L Transistor_BJT:2N3906 Q2
 U 1 1 5C1251E5
 P 6350 3775
@@
 Connection ~ 5850 3775
 $Comp
-L R R6
+L Device:R R6
 U 1 1 5C1254CA
 P 6450 3350
@@
 	6450 3125 6450 3200
 Wire Wire Line
-	5475 3125 6450 3125
-Wire Wire Line
-	5850 3050 5850 3400
+	5475 3125 5850 3125
 Connection ~ 5850 3125
 $Comp
-L R R7
+L Device:R R7
 U 1 1 5C125747
 P 6450 4275
@@
 $EndComp
 Wire Wire Line
-	6450 3975 6450 4125
+	6450 3975 6450 4050
 Connection ~ 6450 4050
 Wire Wire Line
 	6450 4700 6450 4425
 $Comp
-L R R8
+L Device:R R8
 U 1 1 5C12628A
 P 4800 5050
@@
 $EndComp
 $Comp
-L Output J2
+L ports:Output J2
 U 1 1 5C1265F4
 P 7575 4250
@@
 Text Label 6675 5050 0    60   ~ 0
 AUD_OUT
-Connection ~ 6450 4700
 Text Notes 7025 6750 0    60   ~ 0
 Based on composite video modification for Atari 2600 by user simon.plata on AtariAge\nforums. Redesigned PCB to match my VDU projects.
 $Comp
-L Video J1
+L ports:Video J1
 U 1 1 5C129CEB
 P 3925 4150
@@
 	6450 4050 7375 4050
 Wire Wire Line
-	7225 4150 7375 4150
-Wire Wire Line
 	4125 4150 4375 4150
 Wire Wire Line
@@
 	4375 5050 4375 4150
 Wire Wire Line
-	7225 4700 7225 4150
-Wire Wire Line
-	7375 4250 7225 4250
-Connection ~ 7225 4250
-Wire Wire Line
 	7375 4350 7300 4350
 Wire Wire Line
 	7300 4350 7300 5050
+Wire Wire Line
+	4575 4050 4650 4050
+Wire Wire Line
+	5025 4050 5100 4050
+Wire Wire Line
+	5025 4050 5025 4275
+Wire Wire Line
+	5475 4050 5550 4050
+Wire Wire Line
+	5475 4050 5475 4125
+Wire Wire Line
+	5850 4700 5850 4775
+Wire Wire Line
+	5850 4700 6450 4700
+Wire Wire Line
+	5850 3775 5850 3850
+Wire Wire Line
+	5850 3125 6450 3125
+Wire Wire Line
+	5850 3125 5850 3400
+Wire Wire Line
+	6450 4050 6450 4125
+Wire Wire Line
+	5475 3050 5475 3125
+Connection ~ 5475 3125
+$Comp
+L power:GND #PWR?
+U 1 1 60459880
+P 7150 4325
+F 0 "#PWR?" H 7150 4075 50  0001 C CNN
+F 1 "GND" H 7150 4175 50  0000 C CNN
+F 2 "" H 7150 4325 50  0001 C CNN
+F 3 "" H 7150 4325 50  0001 C CNN
+	1    7150 4325
+	1    0    0    -1
+$EndComp
+Wire Wire Line
+	7150 4325 7150 4250
+Connection ~ 7150 4250
+Wire Wire Line
+	7150 4250 7150 4150
+Wire Wire Line
+	7150 4250 7375 4250
+Wire Wire Line
+	7150 4150 7375 4150
 $EndSCHEMATC
